File: IOB_V4.kicad_sch (KiCad schematic)
At the start: 9 parts, among them J1 Conn_01x02, J18 Conn_01x10, J2 Conn_01x03, J20 Conn_01x10, U1 REF3033

Commit message: WIP
Parts:
- added TP4: TestPoint, TestPoint:TestPoint_THTPad_D1.0mm_Drill0.5mm, symbol Connector:TestPoint
Connections:
- net +24V: now also TP4.1
Changed lines of the file:
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@@
     (pin "2")
+  )
+  (symbol (lib_id "Connector:TestPoint") (at 81.661 141.478 0) (unit 1)
+    (in_bom yes) (on_board yes) (fields_autoplaced)
+    (property "Reference" "TP4" (id 0) (at 83.566 138.1759 0)
+      (effects (font (size 1.27 1.27)) (justify left))
+    )
+    (property "Value" "TestPoint" (id 1) (at 80.1878 138.5062 0)
+      (effects (font (size 1.27 1.27)) (justify right) hide)
+    )
+    (property "Footprint" "TestPoint:TestPoint_THTPad_D1.0mm_Drill0.5mm" (id 2) (at 86.741 141.478 0)
+      (effects (font (size 1.27 1.27)) hide)
+    )
+    (property "Datasheet" "~" (id 3) (at 86.741 141.478 0)
+      (effects (font (size 1.27 1.27)) hide)
+    )
+    (pin "1")
   )
   (symbol (lib_id "power:GND") (at 236.982 87.503 0) (unit 1)
@@
       (reference "TP3") (unit 1) (value "TestPoint") (footprint "TestPoint:TestPoint_THTPad_D1.0mm_Drill0.5mm")
     )
-    (path "/534d7b1f-d272-47da-b7a1-47aab2c48175/6a8bea66-9b1e-4f28-aad3-092e91290323"
+    (path "/c42770d1-8453-4584-bf46-7e1cdf558de4"
       (reference "TP4") (unit 1) (value "TestPoint") (footprint "TestPoint:TestPoint_THTPad_D1.0mm_Drill0.5mm")
     )
+    (path "/33332500-4da3-42ef-9bb3-bc804f9ab4ce/53beb16e-3077-404e-84ff-ae3242e55708"
+      (reference "TP5") (unit 1) (value "TestPoint") (footprint "TestPoint:TestPoint_THTPad_D1.0mm_Drill0.5mm")
+    )
     (path "/31b062d9-fa48-4ba2-b857-360e76517386"

Commit message: Annotation fix
Other:
- sheet MCU ports: added ANALOG_IN_0, En0; removed ANALOG_IN_12, En12
- sheet Pressure ports: added Enable0, Out0; removed Enable12, Out12
