File: IOB_V4.kicad_sch (KiCad schematic)
At the start: 10 parts, among them J1 Conn_01x02, J18 Conn_01x10, J2 Conn_01x03, J20 Conn_01x10, U1 REF3033

Commit message: WIP
Parts:
- C2: symbol Device:CP -> Device:C_Polarized
Connections:
- net +3V3 renamed +3.3V

Commit message: Almost ready to be ordered
Parts:
- added G2: Lamarr_Missionpatch, TXV_Library_Footprints:Lamarr_Missionpatch_20x20mm, symbol TXV_Library_Symbols:Lamarr_Missionpatch
- C2: symbol Device:C_Polarized -> Device:CP
Connections:
- net SPI4_NSS8 is gone; now on net SPI4_NSS7: J18.8 (Pin_8)
- net SPI4_NSS1: now also J20.6 (Pin_6); no longer J20.5 (Pin_5)
- net SPI4_NSS2: now also J20.7 (Pin_7); no longer J20.6 (Pin_6)
- net SPI4_NSS3: now also J20.8 (Pin_8); no longer J20.7 (Pin_7)
- net SPI4_NSS4: now also J18.5 (Pin_5); no longer J20.8 (Pin_8)
- net SPI4_NSS5: now also J18.6 (Pin_6); no longer J18.5 (Pin_5)
- net SPI4_NSS6: now also J18.7 (Pin_7); no longer J18.6 (Pin_6)
- net SPI4_NSS7: no longer J18.7 (Pin_7)
- net +3.3V renamed +3V3
- new net SPI4_NSS0: J20.5 (Pin_5)
Other:
- sheet MCU ports: added SPI4_~{CS}0; removed SPI4_~{CS}8

Commit message: Added Servo Config
Parts:
- added J22: Conn_01x02, TXV_Library_Footprints:Molex_Nano-Fit_105309-xx02_1x02_P2.50mm_Vertical, symbol Connector_Generic:Conn_01x02
- added TP6: TestPoint, TestPoint:TestPoint_Loop_D2.54mm_Drill1.5mm_Beaded, symbol Connector:TestPoint
Connections:
- net GND: now also J22.2 (Pin_2)
- new net +12V: J22.1 (Pin_1), TP6.1
