File: pressure_readout.kicad_sch (KiCad schematic)
At the start: 0 parts

Commit message: Annotation fix
Other:
- sheet Input12 renamed Input0
Changed lines of the file:
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@@
     (effects (font (size 1.27 1.27)) (justify left))
   )
-  (hierarchical_label "Out12" (shape output) (at 220.853 115.062 0)
+  (hierarchical_label "Out0" (shape output) (at 220.853 115.062 0)
     (effects (font (size 1.27 1.27)) (justify left))
   )
@@
     (effects (font (size 1.27 1.27)) (justify left))
   )
-  (hierarchical_label "Enable12" (shape bidirectional) (at 220.853 117.221 0)
+  (hierarchical_label "Enable0" (shape bidirectional) (at 220.853 117.221 0)
     (effects (font (size 1.27 1.27)) (justify left))
   )
@@
     (stroke (width 0.1524) (type solid) (color 0 0 0 0))
     (fill (color 0 0 0 0.0000))
-    (property "Sheet name" "Input12" (id 0) (at 193.675 112.4454 0)
+    (property "Sheet name" "Input0" (id 0) (at 193.675 112.4454 0)
       (effects (font (size 1.27 1.27)) (justify left bottom))
     )
