File: pressure_submodule.kicad_sch (KiCad schematic)
At the start: 17 parts, among them IC12 PINA350ABSIDDFR, J14 Conn_01x04, Q12 BSZ0902NSATMA1

Commit message: Correct MUX Footprint added
Parts:
- removed JP72: Jumper_2_Open, Jumper:SolderJumper-2_P1.3mm_Open_TrianglePad1.0x1.5mm, symbol Jumper:Jumper_2_Open
- IC12: footprint SOT65P280X110-8N -> TXV_Library_Footprints:SOT65P280X110-8N
Other:
- note removed: "R2L"
Changed lines of the file:
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@@
   (junction (at 223.52 144.526) (diameter 0) (color 0 0 0 0)
-  )
-  (junction (at 231.14 144.526) (diameter 0) (color 0 0 0 0)
   )
   (junction (at 223.52 114.046) (diameter 0) (color 0 0 0 0)
@@
     (stroke (width 0) (type default) (color 0 0 0 0))
   )
-  (wire (pts (xy 231.14 144.526) (xy 241.3 144.526))
-    (stroke (width 0) (type default) (color 0 0 0 0))
-  )
   (wire (pts (xy 231.14 126.746) (xy 223.52 126.746))
     (stroke (width 0) (type default) (color 0 0 0 0))
@@
     (stroke (width 0) (type default) (color 0 0 0 0))
   )
-  (wire (pts (xy 241.3 133.096) (xy 241.3 131.191))
-    (stroke (width 0) (type default) (color 0 0 0 0))
-  )
   (wire (pts (xy 185.166 94.361) (xy 208.28 94.361))
     (stroke (width 0) (type default) (color 0 0 0 0))
@@
   )
   (wire (pts (xy 212.09 113.411) (xy 212.09 114.046))
-    (stroke (width 0) (type default) (color 0 0 0 0))
-  )
-  (wire (pts (xy 241.3 143.256) (xy 241.3 144.526))
     (stroke (width 0) (type default) (color 0 0 0 0))
   )
@@
     (effects (font (size 1.27 1.27)) (justify left bottom))
   )
-  (text "R2L" (at 243.205 139.446 0)
-    (effects (font (size 1.27 1.27)) (justify left bottom))
-  )
   (text "X" (at 94.869 170.18 0)
     (effects (font (size 1.27 1.27)) (justify left bottom))
@@
     )
     (property "Datasheet" "~" (id 3) (at 181.864 99.441 0)
-      (effects (font (size 1.27 1.27)) hide)
-    )
-    (pin "1")
-    (pin "2")
-  )
-  (symbol (lib_id "Jumper:Jumper_2_Open") (at 241.3 138.176 270)
-    (in_bom yes) (on_board yes)
-    (property "Reference" "JP72" (id 0) (at 237.49 138.176 90)
-      (effects (font (size 1.27 1.27)) (justify left))
-    )
-    (property "Value" "Jumper_2_Open" (id 1) (at 243.7892 139.319 90)
-      (effects (font (size 1.27 1.27)) (justify left) hide)
-    )
-    (property "Footprint" "Jumper:SolderJumper-2_P1.3mm_Open_TrianglePad1.0x1.5mm" (id 2) (at 241.3 138.176 0)
-      (effects (font (size 1.27 1.27)) hide)
-    )
-    (property "Datasheet" "~" (id 3) (at 241.3 138.176 0)
       (effects (font (size 1.27 1.27)) hide)
     )
@@
     (pin "1")
     (pin "2")
-  )
-  (symbol (lib_id "power:+3.3V") (at 241.3 131.191 0)
-    (in_bom yes) (on_board yes)
-    (property "Reference" "#PWR0108" (id 0) (at 241.3 135.001 0)
-      (effects (font (size 1.27 1.27)) hide)
-    )
-    (property "Value" "+3.3V" (id 1) (at 245.11 129.921 0))
-    (property "Footprint" "" (id 2) (at 241.3 131.191 0)
-      (effects (font (size 1.27 1.27)) hide)
-    )
-    (property "Datasheet" "" (id 3) (at 241.3 131.191 0)
-      (effects (font (size 1.27 1.27)) hide)
-    )
-    (pin "1")
   )
   (symbol (lib_id "Device:Polyfuse") (at 213.868 81.28 0)
@@
     (property "Reference" "IC12" (id 0) (at 165.862 79.248 0))
     (property "Value" "PINA350ABSIDDFR" (id 1) (at 165.862 81.788 0))
-    (property "Footprint" "SOT65P280X110-8N" (id 2) (at 155.702 96.901 0)
+    (property "Footprint" "TXV_Library_Footprints:SOT65P280X110-8N" (id 2) (at 155.702 96.901 0)
       (effects (font (size 1.27 1.27)) (justify left) hide)
     )

Commit message: Circuit fix
Parts:
- removed D13: D, Diode_SMD:D_SOD-123F, symbol Device:D
- removed F24: Polyfuse, TXV_Library_Footprints:0805L110SL PPTC Polyfuse Littelfuse, symbol Device:Polyfuse
- removed IC12: PINA350ABSIDDFR, TXV_Library_Footprints:SOT65P280X110-8N, symbol TXV_Library_Symbols:PINA350ABSIDDFR
- removed JP34, JP67, JP68: Jumper_2_Open, Jumper:SolderJumper-2_P1.3mm_Open_TrianglePad1.0x1.5mm, symbol Jumper:Jumper_2_Open
- removed Q12: BSZ0902NSATMA1, TXV_Library_Footprints:PG_TSDSON-8, symbol TXV_Library_Symbols:BSZ0902NSATMA1
- removed R80, R82: R, Resistor_SMD:R_0603_1608Metric, symbol Device:R
- removed R81: Rgate, Resistor_SMD:R_0603_1608Metric, symbol Device:R
- removed R83, R84: Rpull, Resistor_SMD:R_0603_1608Metric, symbol Device:R
- added 160R?: 160R, Resistor_SMD:R_0603_1608Metric, symbol Device:R
- added C? (x2): C, symbol Device:C
- added C?: (no value), symbol Device:C
- added D? (x3): D, Diode_SMD:D_SOD-123F, symbol Device:D
- added F? (x7): Polyfuse, TXV_Library_Footprints:0805L110SL PPTC Polyfuse Littelfuse, symbol Device:Polyfuse
- added IC? (x4): PINA350ABSIDDFR, TXV_Library_Footprints:SOT65P280X110-8N, symbol TXV_Library_Symbols:PINA350ABSIDDFR
- added J? (x5): Conn_01x04, TXV_Library_Footprints:TE_M12_4_Pin_PCB, symbol Connector_Generic:Conn_01x04
- added JP? (x16): Jumper_2_Open, Jumper:SolderJumper-2_P1.3mm_Open_TrianglePad1.0x1.5mm, symbol Jumper:Jumper_2_Open
- added Q? (x3): BSZ0902NSATMA1, TXV_Library_Footprints:PG_TSDSON-8, symbol TXV_Library_Symbols:BSZ0902NSATMA1
- added R? (x4): (no value), Resistor_SMD:R_0603_1608Metric, symbol Device:R
- added R? (x3): NP, Resistor_SMD:R_0603_1608Metric, symbol Device:R
- added R? (x2): 100m, Resistor_SMD:R_0603_1608Metric, symbol Device:R
- added R? (x2): Rpull, Resistor_SMD:R_0603_1608Metric, symbol Device:R
- added R? (x3): Rgate, Resistor_SMD:R_0603_1608Metric, symbol Device:R
- added R? (x3): 0R, Resistor_SMD:R_0603_1608Metric, symbol Device:R
- added R?: R, Resistor_SMD:R_0603_1608Metric, symbol Device:R
- renumbered F23 to F1, J14 to J3, R78 to R1, R79 to R2
Connections:
- net +24V: now also F?.1, F?.1, F?.1, F?.1
- net +3V3: now also F?.1, F?.1, F?.1, IC?.7 (V+), IC?.7 (V+), IC?.7 (V+), IC?.7 (V+)
- net AnalogOut: now also C?.1, C?.1, C?.1, IC?.6 (OUT), R?.1, R?.1, R?.1, R?.1, R?.2
- net Enable-Selection1: now also R?.1, R?.1, R?.1
- net GND: now also J3.4 (Pin_4), 160R?.2, C?.2, C?.2, C?.2, D?.2 (A), D?.2 (A), IC?.2 (IN-), IC?.4 (V-), IC?.4 (V-), IC?.4 (V-), IC?.4 (V-), IC?.5 (REF), IC?.5 (REF), IC?.5 (REF), IC?.5 (REF), J?.4 (Pin_4), JP?.1 (A), JP?.1 (A), JP?.1 (A), JP?.1 (A), JP?.1 (A), JP?.1 (A), JP?.1 (A), JP?.2 (B), R?.2, R?.2, R?.2, R?.2, R?.2, R?.2, R?.2
- net at J3.2 (Pin_2): now also J3.3 (Pin_3), R1.1
- new net: F?.2, J?.1 (Pin_1) (x3)
- new net: 160R?.1, J?.2 (Pin_2), J?.3 (Pin_3), R?.2
- new net: IC?.3 (IN+), Q?.1 (S), R?.1
- new net: Q?.2 (G), R?.1, R?.2 (x3)
- new net: D?.1 (K), J?.2 (Pin_2), Q?.3 (D)
- new net: IC?.6 (OUT), JP?.1 (A), R?.1 (x2)
- new net: D?.1 (K), J?.2 (Pin_2), JP?.2 (B), JP?.2 (B), JP?.2 (B), Q?.3 (D) (x2)
- new net: R?.1, R?.2, R?.2 (x2)
- new net: IC?.3 (IN+), JP?.1 (A), Q?.1 (S), R?.1 (x2)
- new net: F?.2, F?.2, J?.1 (Pin_1) (x2)
- new net: J?.3 (Pin_3), JP?.1 (A), JP?.2 (B) (x2)
- new net: IC?.1 (GS), JP?.2 (B) (x4)
- new net: IC?.6 (OUT), R?.1
- new net: IC?.3 (IN+), J?.2 (Pin_2)
- new net: IC?.2 (IN-), J?.3 (Pin_3)
- new net: IC?.2 (IN-), JP?.1 (A), JP?.1 (A)
- new net: D?.2 (A), IC?.2 (IN-), JP?.1 (A), JP?.2 (B), R?.2, R?.2
- new net: J?.4 (Pin_4), JP?.2 (B) (x2)
- no-connect marks 1 -> 7
Other:
- note added: "10k oder 0"
- note added: "4 - 20 mA"
- note added: "Bridge"
- note added: "Digital Out"
- note added: "Digital/Analog In"
- note removed: "JF"
- note removed: "JO"
- note removed: "R1U"
- note removed: "RG"
- moved on the sheet: F1, J3, R1, R2

Commit message: WIP
Parts:
- removed C?: C, symbol Device:C
- removed D?: D, Diode_SMD:D_SOD-123F, symbol Device:D
- removed F? (x2): Polyfuse, TXV_Library_Footprints:0805L110SL PPTC Polyfuse Littelfuse, symbol Device:Polyfuse
- removed IC?: PINA350ABSIDDFR, TXV_Library_Footprints:SOT65P280X110-8N, symbol TXV_Library_Symbols:PINA350ABSIDDFR
- removed J?: Conn_01x04, TXV_Library_Footprints:TE_M12_4_Pin_PCB, symbol Connector_Generic:Conn_01x04
- removed JP? (x7): Jumper_2_Open, Jumper:SolderJumper-2_P1.3mm_Open_TrianglePad1.0x1.5mm, symbol Jumper:Jumper_2_Open
- removed Q?: BSZ0902NSATMA1, TXV_Library_Footprints:PG_TSDSON-8, symbol TXV_Library_Symbols:BSZ0902NSATMA1
- removed R?: Rpull, Resistor_SMD:R_0603_1608Metric, symbol Device:R
- removed R?: (no value), Resistor_SMD:R_0603_1608Metric, symbol Device:R
- removed R?: NP, Resistor_SMD:R_0603_1608Metric, symbol Device:R
- removed R?: Rgate, Resistor_SMD:R_0603_1608Metric, symbol Device:R
- removed R?: 0R, Resistor_SMD:R_0603_1608Metric, symbol Device:R
- removed R?: 100m, Resistor_SMD:R_0603_1608Metric, symbol Device:R
Connections:
- no-connect marks 7 -> 6
Other:
- moved on the sheet: C?, D?, F?, IC?, J?, JP?, Q?, R?

Commit message: Annotation fix
Parts:
- removed 160R?: 160R, Resistor_SMD:R_0603_1608Metric, symbol Device:R
- removed C?: (no value), symbol Device:C
- removed D?: D, Diode_SMD:D_SOD-123F, symbol Device:D
- removed F1, F? (x3): Polyfuse, TXV_Library_Footprints:0805L110SL PPTC Polyfuse Littelfuse, symbol Device:Polyfuse
- removed IC? (x2): PINA350ABSIDDFR, TXV_Library_Footprints:SOT65P280X110-8N, symbol TXV_Library_Symbols:PINA350ABSIDDFR
- removed J3, J? (x3): Conn_01x04, TXV_Library_Footprints:TE_M12_4_Pin_PCB, symbol Connector_Generic:Conn_01x04
- removed JP? (x2): Jumper_2_Open, Jumper:SolderJumper-2_P1.3mm_Open_TrianglePad1.0x1.5mm, symbol Jumper:Jumper_2_Open
- removed Q?: BSZ0902NSATMA1, TXV_Library_Footprints:PG_TSDSON-8, symbol TXV_Library_Symbols:BSZ0902NSATMA1
- removed R1, R?: 0R, Resistor_SMD:R_0603_1608Metric, symbol Device:R
- removed R2, R?: NP, Resistor_SMD:R_0603_1608Metric, symbol Device:R
- removed R? (x3): (no value), Resistor_SMD:R_0603_1608Metric, symbol Device:R
- removed R?: Rgate, Resistor_SMD:R_0603_1608Metric, symbol Device:R
- C20: renamed from C?; footprint (none) -> Capacitor_SMD:C_0603_1608Metric
- gave numbers to parts that had none: 19
Connections:
- no-connect marks 6 -> 1
Other:
- note added: "0"
- note added: "0,1"
- note added: "10k"
- note added: "160"
- note added: "4-20mA IN: J24V, JO, RG=160R, A coding dig/anaIn: JO, J3V3, RFU, D coding powerOut: J24V, FET, RFL, RS=shunt, JF, B coding"
- note added: "F3V3 F24V J1 J2 J3 J4 J5 J6 FET INA C RO R1H R1L RG R2L RS Pinout ChannelType"
- note added: "J1"
- note added: "J2"
- note added: "J3"
- note added: "J4"
- note added: "J5"
- note added: "J6"
- note added: "R1H"
- note added: "R2L"
- note added: "RG"
- note added: "RO"
- note added: "RS"
- note added: "pwr 1 in 2-3 gnd 4"
- note removed: "10k oder 0"
- note removed: "4 - 20 mA"
- note removed: "4-20mA IN: J24V, JO, RG=160R, A coding dig/anaIn: JO, J3V3, RFU, D coding powerOut: J24V, FET, RFL, RI=shunt, JF, B coding"
- note removed: "Digital Out"
- note removed: "Digital/Analog In"
- note removed: "F3V3 F24V RI RG R1U R1L R2U R2L JO INA JF FET Pinout ChannelType"
- note removed: "RI"
- moved on the sheet: C20, D2, F1, F2, IC1, J3, JP1, JP2, JP3, JP4, JP5, JP6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

Commit message: Footprint separation
Parts:
- renumbered C20 to C31, D2 to D13, F1 to F23, F2 to F24, IC1 to IC12, J3 to J14, JP1 to JP78, JP2 to JP79, JP3 to JP80, JP4 to JP81, JP5 to JP82, JP6 to JP83, JP7 to JP84, Q1 to Q12, R1 to R67, R2 to R68, R3 to R69, R4 to R70, R5 to R71, R6 to R72
Changed lines of the file:
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@@
   (symbol (lib_id "power:GND") (at 204.216 77.343 0)
     (in_bom yes) (on_board yes) (fields_autoplaced)
-    (property "Reference" "#PWR019" (id 0) (at 204.216 83.693 0)
+    (property "Reference" "#PWR096" (id 0) (at 204.216 83.693 0)
       (effects (font (size 1.27 1.27)) hide)
     )
@@
   (symbol (lib_id "power:+3.3V") (at 67.564 80.899 0)
     (in_bom yes) (on_board yes)
-    (property "Reference" "#PWR014" (id 0) (at 67.564 84.709 0)
+    (property "Reference" "#PWR091" (id 0) (at 67.564 84.709 0)
       (effects (font (size 1.27 1.27)) hide)
     )
@@
   (symbol (lib_id "Device:R") (at 55.372 105.41 0)
     (in_bom yes) (on_board yes)
-    (property "Reference" "R3" (id 0) (at 51.562 105.283 0)
+    (property "Reference" "R69" (id 0) (at 51.562 105.283 0)
       (effects (font (size 1.27 1.27)) (justify left))
     )
@@
   (symbol (lib_id "TXV_Library_Symbols:BSZ0902NSATMA1") (at 162.052 74.549 0)
     (in_bom yes) (on_board yes)
-    (property "Reference" "Q1" (id 0) (at 165.989 74.549 0)
+    (property "Reference" "Q12" (id 0) (at 165.989 74.549 0)
       (effects (font (size 1.27 1.27)) (justify left))
     )
@@
   (symbol (lib_id "power:GND") (at 55.372 110.49 0)
     (in_bom yes) (on_board yes) (fields_autoplaced)
-    (property "Reference" "#PWR013" (id 0) (at 55.372 116.84 0)
+    (property "Reference" "#PWR090" (id 0) (at 55.372 116.84 0)
       (effects (font (size 1.27 1.27)) hide)
     )
@@
   (symbol (lib_id "Jumper:Jumper_2_Open") (at 191.008 63.373 90)
     (in_bom yes) (on_board yes)
-    (property "Reference" "JP5" (id 0) (at 187.833 64.643 0)
+    (property "Reference" "JP82" (id 0) (at 187.833 64.643 0)
       (effects (font (size 1.27 1.27)) (justify left))
     )
@@
   (symbol (lib_id "power:+3.3V") (at 200.152 44.069 0)
     (in_bom yes) (on_board yes)
-    (property "Reference" "#PWR018" (id 0) (at 200.152 47.879 0)
+    (property "Reference" "#PWR095" (id 0) (at 200.152 47.879 0)
       (effects (font (size 1.27 1.27)) hide)
     )
@@
   (symbol (lib_id "power:GND") (at 109.855 107.188 0)
     (in_bom yes) (on_board yes) (fields_autoplaced)
-    (property "Reference" "#PWR015" (id 0) (at 109.855 113.538 0)
+    (property "Reference" "#PWR092" (id 0) (at 109.855 113.538 0)
       (effects (font (size 1.27 1.27)) hide)
     )
@@
   (symbol (lib_id "Device:Polyfuse") (at 186.182 49.403 0)
     (in_bom yes) (on_board yes) (fields_autoplaced)
-    (property "Reference" "F1" (id 0) (at 188.595 48.1329 0)
+    (property "Reference" "F23" (id 0) (at 188.595 48.1329 0)
       (effects (font (size 1.27 1.27)) (justify left))
     )
@@
   (symbol (lib_id "TXV_Library_Symbols:PINA350ABSIDDFR") (at 99.822 92.075 180)
     (in_bom yes) (on_board yes) (fields_autoplaced)
-    (property "Reference" "IC1" (id 0) (at 85.852 76.962 0))
+    (property "Reference" "IC12" (id 0) (at 85.852 76.962 0))
     (property "Value" "PINA350ABSIDDFR" (id 1) (at 85.852 79.502 0))
     (property "Footprint" "TXV_Library_Footprints:SOT65P280X110-8N" (id 2) (at 75.692 94.615 0)
@@
   (symbol (lib_id "Jumper:Jumper_2_Open") (at 101.854 97.155 90)
     (in_bom yes) (on_board yes)
-    (property "Reference" "JP1" (id 0) (at 98.679 98.425 0)
+    (property "Reference" "JP78" (id 0) (at 98.679 98.425 0)
       (effects (font (size 1.27 1.27)) (justify left))
     )
@@
   (symbol (lib_id "Device:R") (at 163.322 91.567 0)
     (in_bom yes) (on_board yes)
-    (property "Reference" "R6" (id 0) (at 158.242 90.297 0)
+    (property "Reference" "R72" (id 0) (at 158.242 90.297 0)
       (effects (font (size 1.27 1.27)) (justify left))
     )
@@
   (symbol (lib_id "Device:C") (at 43.434 105.283 0)
     (in_bom yes) (on_board yes)
-    (property "Reference" "C20" (id 0) (at 39.37 103.505 0)
+    (property "Reference" "C31" (id 0) (at 39.37 103.505 0)
       (effects (font (size 1.27 1.27)) (justify left))
     )
@@
   (symbol (lib_id "Jumper:Jumper_2_Open") (at 191.008 73.533 90)
     (in_bom yes) (on_board yes)
-    (property "Reference" "JP6" (id 0) (at 187.833 74.803 0)
+    (property "Reference" "JP83" (id 0) (at 187.833 74.803 0)
       (effects (font (size 1.27 1.27)) (justify left))
     )
@@
   (symbol (lib_id "Jumper:Jumper_2_Open") (at 143.256 89.535 0)
     (in_bom yes) (on_board yes)
-    (property "Reference" "JP4" (id 0) (at 141.986 86.36 0)
+    (property "Reference" "JP81" (id 0) (at 141.986 86.36 0)
       (effects (font (size 1.27 1.27)) (justify left))
     )
@@
   (symbol (lib_id "Device:R") (at 143.637 74.549 90)
     (in_bom yes) (on_board yes)
-    (property "Reference" "R4" (id 0) (at 143.002 72.644 90)
+    (property "Reference" "R70" (id 0) (at 143.002 72.644 90)
       (effects (font (size 1.27 1.27)) (justify left))
     )
@@
   (symbol (lib_id "Jumper:Jumper_2_Open") (at 106.172 58.293 0)
     (in_bom yes) (on_board yes)
-    (property "Reference" "JP2" (id 0) (at 104.902 55.118 0)
+    (property "Reference" "JP79" (id 0) (at 104.902 55.118 0)
       (effects (font (size 1.27 1.27)) (justify left))
     )
@@
   (symbol (lib_id "Jumper:Jumper_2_Open") (at 113.03 64.643 90)
     (in_bom yes) (on_board yes)
-    (property "Reference" "JP3" (id 0) (at 109.855 65.913 0)
+    (property "Reference" "JP80" (id 0) (at 109.855 65.913 0)
       (effects (font (size 1.27 1.27)) (justify left))
     )
@@
   (symbol (lib_id "Device:D") (at 170.942 73.914 270)
     (in_bom yes) (on_board yes)
-    (property "Reference" "D2" (id 0) (at 172.9486 72.7456 90)
+    (property "Reference" "D13" (id 0) (at 172.9486 72.7456 90)
       (effects (font (size 1.27 1.27)) (justify left))
     )
@@
   (symbol (lib_id "power:+24V") (at 186.182 44.069 0)
     (in_bom yes) (on_board yes)
-    (property "Reference" "#PWR017" (id 0) (at 186.182 47.879 0)
+    (property "Reference" "#PWR094" (id 0) (at 186.182 47.879 0)
       (effects (font (size 1.27 1.27)) hide)
     )
@@
   (symbol (lib_id "Device:Polyfuse") (at 200.152 49.403 0)
     (in_bom yes) (on_board yes) (fields_autoplaced)
-    (property "Reference" "F2" (id 0) (at 202.565 48.1329 0)
+    (property "Reference" "F24" (id 0) (at 202.565 48.1329 0)
       (effects (font (size 1.27 1.27)) (justify left))
     )
@@
   (symbol (lib_id "Connector_Generic:Conn_01x04") (at 213.106 58.293 0)
     (in_bom yes) (on_board yes)
-    (property "Reference" "J3" (id 0) (at 215.138 58.4962 0)
+    (property "Reference" "J14" (id 0) (at 215.138 58.4962 0)
       (effects (font (size 1.27 1.27)) (justify left))
     )
@@
   (symbol (lib_id "power:GND") (at 163.322 103.505 0)
     (in_bom yes) (on_board yes) (fields_autoplaced)
-    (property "Reference" "#PWR016" (id 0) (at 163.322 109.855 0)
+    (property "Reference" "#PWR093" (id 0) (at 163.322 109.855 0)
       (effects (font (size 1.27 1.27)) hide)
     )
@@
   (symbol (lib_id "Device:R") (at 151.892 79.629 0)
     (in_bom yes) (on_board yes)
-    (property "Reference" "R5" (id 0) (at 145.542 78.359 0)
+    (property "Reference" "R71" (id 0) (at 145.542 78.359 0)
       (effects (font (size 1.27 1.27)) (justify left))
     )
@@
   (symbol (lib_id "Device:R") (at 55.372 95.25 0)
     (in_bom yes) (on_board yes)
-    (property "Reference" "R2" (id 0) (at 50.292 93.345 0)
+    (property "Reference" "R68" (id 0) (at 50.292 93.345 0)
       (effects (font (size 1.27 1.27)) (justify left))
     )
@@
   (symbol (lib_id "Jumper:Jumper_2_Open") (at 204.216 69.977 90)
     (in_bom yes) (on_board yes)
-    (property "Reference" "JP7" (id 0) (at 201.041 71.247 0)
+    (property "Reference" "JP84" (id 0) (at 201.041 71.247 0)
       (effects (font (size 1.27 1.27)) (justify left))
     )
@@
   (symbol (lib_id "Device:R") (at 49.53 100.457 90)
     (in_bom yes) (on_board yes)
-    (property "Reference" "R1" (id 0) (at 50.292 102.489 90)
-      (effects (font (size 1.27 1.27)) (justify left))
-    )
+    (property "Reference" "R67" (id 0) (at 50.292 102.489 90)
+      (effects (font (size 1.27 1.27)) (justify left))
+    )
