File: pressure_submodule.kicad_sch (KiCad schematic)
At the start: 20 parts, among them IC12 PINA350ABSIDDFR, J14 Conn_01x04, Q12 BSZ0902NSATMA1

Commit message: WIP
Parts:
- renumbered C31 to C30, D13 to D12, F23 to F21, F24 to F22, IC12 to IC11, J14 to J13, JP78 to JP71, JP79 to JP72, JP80 to JP73, JP81 to JP74, JP82 to JP75, JP83 to JP76, JP84 to JP77, Q12 to Q11, R67 to R61, R68 to R62, R69 to R63, R70 to R64, R71 to R65, R72 to R66
Changed lines of the file:
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@@
   (symbol (lib_id "Device:R") (at 55.372 105.41 0)
     (in_bom yes) (on_board yes)
-    (property "Reference" "R69" (id 0) (at 51.562 105.283 0)
+    (property "Reference" "R63" (id 0) (at 51.562 105.283 0)
       (effects (font (size 1.27 1.27)) (justify left))
     )
@@
   (symbol (lib_id "TXV_Library_Symbols:BSZ0902NSATMA1") (at 162.052 74.549 0)
     (in_bom yes) (on_board yes)
-    (property "Reference" "Q12" (id 0) (at 165.989 74.549 0)
+    (property "Reference" "Q11" (id 0) (at 165.989 74.549 0)
       (effects (font (size 1.27 1.27)) (justify left))
     )
@@
   (symbol (lib_id "Jumper:Jumper_2_Open") (at 191.008 63.373 90)
     (in_bom yes) (on_board yes)
-    (property "Reference" "JP82" (id 0) (at 187.833 64.643 0)
+    (property "Reference" "JP75" (id 0) (at 187.833 64.643 0)
       (effects (font (size 1.27 1.27)) (justify left))
     )
@@
   (symbol (lib_id "Device:Polyfuse") (at 186.182 49.403 0)
     (in_bom yes) (on_board yes) (fields_autoplaced)
-    (property "Reference" "F23" (id 0) (at 188.595 48.1329 0)
+    (property "Reference" "F21" (id 0) (at 188.595 48.1329 0)
       (effects (font (size 1.27 1.27)) (justify left))
     )
@@
   (symbol (lib_id "TXV_Library_Symbols:PINA350ABSIDDFR") (at 99.822 92.075 180)
     (in_bom yes) (on_board yes) (fields_autoplaced)
-    (property "Reference" "IC12" (id 0) (at 85.852 76.962 0))
+    (property "Reference" "IC11" (id 0) (at 85.852 76.962 0))
     (property "Value" "PINA350ABSIDDFR" (id 1) (at 85.852 79.502 0))
     (property "Footprint" "TXV_Library_Footprints:SOT65P280X110-8N" (id 2) (at 75.692 94.615 0)
@@
   (symbol (lib_id "Jumper:Jumper_2_Open") (at 101.854 97.155 90)
     (in_bom yes) (on_board yes)
-    (property "Reference" "JP78" (id 0) (at 98.679 98.425 0)
+    (property "Reference" "JP71" (id 0) (at 98.679 98.425 0)
       (effects (font (size 1.27 1.27)) (justify left))
     )
@@
   (symbol (lib_id "Device:R") (at 163.322 91.567 0)
     (in_bom yes) (on_board yes)
-    (property "Reference" "R72" (id 0) (at 158.242 90.297 0)
+    (property "Reference" "R66" (id 0) (at 158.242 90.297 0)
       (effects (font (size 1.27 1.27)) (justify left))
     )
@@
   (symbol (lib_id "Device:C") (at 43.434 105.283 0)
     (in_bom yes) (on_board yes)
-    (property "Reference" "C31" (id 0) (at 39.37 103.505 0)
+    (property "Reference" "C30" (id 0) (at 39.37 103.505 0)
       (effects (font (size 1.27 1.27)) (justify left))
     )
@@
   (symbol (lib_id "Jumper:Jumper_2_Open") (at 191.008 73.533 90)
     (in_bom yes) (on_board yes)
-    (property "Reference" "JP83" (id 0) (at 187.833 74.803 0)
+    (property "Reference" "JP76" (id 0) (at 187.833 74.803 0)
       (effects (font (size 1.27 1.27)) (justify left))
     )
@@
   (symbol (lib_id "Jumper:Jumper_2_Open") (at 143.256 89.535 0)
     (in_bom yes) (on_board yes)
-    (property "Reference" "JP81" (id 0) (at 141.986 86.36 0)
+    (property "Reference" "JP74" (id 0) (at 141.986 86.36 0)
       (effects (font (size 1.27 1.27)) (justify left))
     )
@@
   (symbol (lib_id "Device:R") (at 143.637 74.549 90)
     (in_bom yes) (on_board yes)
-    (property "Reference" "R70" (id 0) (at 143.002 72.644 90)
+    (property "Reference" "R64" (id 0) (at 143.002 72.644 90)
       (effects (font (size 1.27 1.27)) (justify left))
     )
@@
   (symbol (lib_id "Jumper:Jumper_2_Open") (at 106.172 58.293 0)
     (in_bom yes) (on_board yes)
-    (property "Reference" "JP79" (id 0) (at 104.902 55.118 0)
+    (property "Reference" "JP72" (id 0) (at 104.902 55.118 0)
       (effects (font (size 1.27 1.27)) (justify left))
     )
@@
   (symbol (lib_id "Jumper:Jumper_2_Open") (at 113.03 64.643 90)
     (in_bom yes) (on_board yes)
-    (property "Reference" "JP80" (id 0) (at 109.855 65.913 0)
+    (property "Reference" "JP73" (id 0) (at 109.855 65.913 0)
       (effects (font (size 1.27 1.27)) (justify left))
     )
@@
   (symbol (lib_id "Device:D") (at 170.942 73.914 270)
     (in_bom yes) (on_board yes)
-    (property "Reference" "D13" (id 0) (at 172.9486 72.7456 90)
+    (property "Reference" "D12" (id 0) (at 172.9486 72.7456 90)
       (effects (font (size 1.27 1.27)) (justify left))
     )
@@
   (symbol (lib_id "Device:Polyfuse") (at 200.152 49.403 0)
     (in_bom yes) (on_board yes) (fields_autoplaced)
-    (property "Reference" "F24" (id 0) (at 202.565 48.1329 0)
+    (property "Reference" "F22" (id 0) (at 202.565 48.1329 0)
       (effects (font (size 1.27 1.27)) (justify left))
     )
@@
   (symbol (lib_id "Connector_Generic:Conn_01x04") (at 213.106 58.293 0)
     (in_bom yes) (on_board yes)
-    (property "Reference" "J14" (id 0) (at 215.138 58.4962 0)
+    (property "Reference" "J13" (id 0) (at 215.138 58.4962 0)
       (effects (font (size 1.27 1.27)) (justify left))
     )
@@
   (symbol (lib_id "Device:R") (at 151.892 79.629 0)
     (in_bom yes) (on_board yes)
-    (property "Reference" "R71" (id 0) (at 145.542 78.359 0)
+    (property "Reference" "R65" (id 0) (at 145.542 78.359 0)
       (effects (font (size 1.27 1.27)) (justify left))
     )
@@
   (symbol (lib_id "Device:R") (at 55.372 95.25 0)
     (in_bom yes) (on_board yes)
-    (property "Reference" "R68" (id 0) (at 50.292 93.345 0)
+    (property "Reference" "R62" (id 0) (at 50.292 93.345 0)
       (effects (font (size 1.27 1.27)) (justify left))
     )
@@
   (symbol (lib_id "Jumper:Jumper_2_Open") (at 204.216 69.977 90)
     (in_bom yes) (on_board yes)
-    (property "Reference" "JP84" (id 0) (at 201.041 71.247 0)
+    (property "Reference" "JP77" (id 0) (at 201.041 71.247 0)
       (effects (font (size 1.27 1.27)) (justify left))
     )
@@
   (symbol (lib_id "Device:R") (at 49.53 100.457 90)
     (in_bom yes) (on_board yes)
-    (property "Reference" "R67" (id 0) (at 50.292 102.489 90)
-      (effects (font (size 1.27 1.27)) (justify left))
-    )
+    (property "Reference" "R61" (id 0) (at 50.292 102.489 90)
+      (effects (font (size 1.27 1.27)) (justify left))
+    )
