File: MCU.kicad_sch (KiCad schematic)
At the start: 44 parts, among them J15 Conn_01x08, J16 Conn_02x04_Odd_Even, J17 Conn_01x04, J19 Conn_01x04, Q13 BSZ0902NSATMA1, SW1 SW_Push_Dual, SW2 SW_Push_Dual, SW3 SW_DIP_x08, U15 MCP1700-3302E_SOT23, U17 MCP2562FD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

Commit message: Connector layout V1
1 of the channels has been set
Connections:
- net ANALOG_IN_0: now also U19.56 (PA8); no longer U19.22 (PC4)
Changed lines of the file:
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@@
   (no_connect (at 128.143 269.875))
   (no_connect (at 316.23 71.882))
-  (no_connect (at 245.11 129.032))
   (no_connect (at 47.625 123.825))
   (no_connect (at 245.11 169.672))
@@
   (no_connect (at 316.23 126.492))
   (no_connect (at 58.293 85.979))
+  (no_connect (at 316.23 103.632))
   (wire (pts (xy 49.403 157.607) (xy 51.943 157.607))
     (stroke (width 0) (type default) (color 0 0 0 0))
@@
     (stroke (width 0) (type default) (color 0 0 0 0))
   )
+  (wire (pts (xy 231.14 129.032) (xy 245.11 129.032))
+    (stroke (width 0) (type default) (color 0 0 0 0))
+  )
   (wire (pts (xy 46.228 264.668) (xy 46.228 273.558))
     (stroke (width 0) (type default) (color 0 0 0 0))
@@
     (stroke (width 0) (type default) (color 0 0 0 0))
   )
-  (wire (pts (xy 330.2 103.632) (xy 316.23 103.632))
-    (stroke (width 0) (type default) (color 0 0 0 0))
-  )
   (wire (pts (xy 266.7 57.658) (xy 266.7 60.452))
     (stroke (width 0) (type default) (color 0 0 0 0))
@@
     (effects (font (size 1.27 1.27)) (justify right bottom))
   )
-  (label "ADC2_IN5" (at 372.618 82.804 0)
+  (label "ADC5_IN1" (at 372.618 82.804 0)
     (effects (font (size 1.27 1.27)) (justify left bottom))
   )
@@
     (effects (font (size 1.27 1.27)) (justify left bottom))
   )
-  (label "ADC5_IN1" (at 372.618 54.991 0)
+  (label "ADC5_IN2" (at 372.618 54.991 0)
+    (effects (font (size 1.27 1.27)) (justify left bottom))
+  )
+  (label "ADC5_IN1" (at 231.14 129.032 0)
     (effects (font (size 1.27 1.27)) (justify left bottom))
   )
@@
     (effects (font (size 1.27 1.27)) (justify left bottom))
   )
-  (label "ADC2_IN5" (at 330.2 103.632 180)
-    (effects (font (size 1.27 1.27)) (justify right bottom))
-  )
   (label "SPI4_NSS" (at 175.006 155.956 180)
     (effects (font (size 1.27 1.27)) (justify right bottom))
@@
     (effects (font (size 1.27 1.27)) (justify right bottom))
   )
-  (label "ADC5_IN1" (at 231.14 131.572 0)
-    (effects (font (size 1.27 1.27)) (justify left bottom))
-  )
+  (label "ADC5_IN2" (at 231.14 131.572 0)
+    (effects (font (size 1.27 1.27)) (justify left bottom))
+  )

Commit message: WIP
Connections:
- net ANALOG_IN_2: now also U19.19 (PA5); no longer U19.48 (PD9)
- net ANALOG_IN_4: now also U19.48 (PD9); no longer U19.19 (PA5)
- net En1: now also U19.54 (PC8); no longer U19.58 (PA10)
- net En2: now also U19.58 (PA10); no longer U19.54 (PC8)
- net En4: now also U19.52 (PC6); no longer U19.65 (PA15)
- net En5: now also U19.65 (PA15); no longer U19.52 (PC6)
Other:
- note removed: "umsetzen"
Changed lines of the file:
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@@
     (stroke (width 0) (type default) (color 0 0 0 0))
   )
-  (text "umsetzen" (at 362.204 82.804 0)
-    (effects (font (size 1.27 1.27)) (justify left bottom))
-  )
   (label "MUX1_SEL2" (at 172.212 171.196 180)
     (effects (font (size 1.27 1.27)) (justify right bottom))
@@
     (effects (font (size 1.27 1.27)) (justify left bottom))
   )
-  (label "En4" (at 231.14 146.812 0)
+  (label "En5" (at 231.14 146.812 0)
     (effects (font (size 1.27 1.27)) (justify left bottom))
   )
@@
     (effects (font (size 1.27 1.27)) (justify right bottom))
   )
-  (label "ADC5_IN13" (at 372.618 57.531 0)
+  (label "ADC2_IN13" (at 372.618 57.531 0)
     (effects (font (size 1.27 1.27)) (justify left bottom))
   )
@@
     (effects (font (size 1.27 1.27)) (justify left bottom))
   )
-  (label "En2" (at 330.2 113.792 180)
+  (label "En1" (at 330.2 113.792 180)
     (effects (font (size 1.27 1.27)) (justify right bottom))
   )
@@
     (effects (font (size 1.27 1.27)) (justify right bottom))
   )
-  (label "ADC2_IN13" (at 372.618 62.611 0)
+  (label "ADC5_IN13" (at 372.618 62.611 0)
     (effects (font (size 1.27 1.27)) (justify left bottom))
   )
@@
     (effects (font (size 1.27 1.27)) (justify left bottom))
   )
-  (label "En1" (at 231.14 134.112 0)
+  (label "En2" (at 231.14 134.112 0)
     (effects (font (size 1.27 1.27)) (justify left bottom))
   )
@@
     (effects (font (size 1.27 1.27)) (justify right bottom))
   )
-  (label "En5" (at 328.93 108.712 180)
-    (effects (font (size 1.27 1.27)) (justify right bottom))
-  )
+  (label "En4" (at 328.93 108.712 180)
+    (effects (font (size 1.27 1.27)) (justify right bottom))
+  )

Commit message: WIP
Connections:
- net ANALOG_IN_0: now also U19.48 (PD9); no longer U19.56 (PA8)
- net ANALOG_IN_3: now also U19.30 (PE7); no longer U19.26 (PB2)
- net ANALOG_IN_4: now also U19.49 (PD10); no longer U19.48 (PD9)
- net ANALOG_IN_5: now also U19.56 (PA8); no longer U19.49 (PD10)
- net ANALOG_IN_6: now also U19.20 (PA6); no longer U19.30 (PE7)
- net ANALOG_IN_7: now also U19.17 (PA3); no longer U19.8 (PC0)
- net ANALOG_IN_8: now also U19.8 (PC0); no longer U19.17 (PA3)
- net ANALOG_IN_9: now also U19.13 (PA1); no longer U19.23 (PC5)
- net En0: now also U19.47 (PD8); no longer U19.12 (PA0)
- net En3: now also U19.26 (PB2); no longer U19.47 (PD8)
- net En6: now also U19.23 (PC5); no longer U19.20 (PA6)
- net En7: now also U19.18 (PA4); no longer U19.71 (PD2)
- net En8: now also U19.71 (PD2); no longer U19.13 (PA1)
- net En9: now also U19.12 (PA0); no longer U19.18 (PA4)
Changed lines of the file:
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@@
-    (stroke (width 0) (type default) (color 0 0 0 0))
-  )
-  (wire (pts (xy 231.14 123.952) (xy 245.11 123.952))
     (stroke (width 0) (type default) (color 0 0 0 0))
   )
@@
     (stroke (width 0) (type default) (color 0 0 0 0))
   )
-  (wire (pts (xy 330.2 106.172) (xy 316.23 106.172))
-    (stroke (width 0) (type default) (color 0 0 0 0))
-  )
   (wire (pts (xy 227.33 113.792) (xy 245.11 113.792))
     (stroke (width 0) (type default) (color 0 0 0 0))
@@
     (stroke (width 0) (type default) (color 0 0 0 0))
   )
+  (wire (pts (xy 316.23 106.172) (xy 330.2 106.172))
+    (stroke (width 0) (type default) (color 0 0 0 0))
+  )
   (wire (pts (xy 133.096 185.42) (xy 135.636 183.896))
     (stroke (width 0) (type default) (color 0 0 0 0))
@@
     (stroke (width 0) (type default) (color 0 0 0 0))
   )
+  (wire (pts (xy 231.14 159.512) (xy 245.11 159.512))
+    (stroke (width 0) (type default) (color 0 0 0 0))
+  )
   (wire (pts (xy 147.828 51.435) (xy 150.749 51.435))
     (stroke (width 0) (type default) (color 0 0 0 0))
@@
     (stroke (width 0) (type default) (color 0 0 0 0))
   )
+  (wire (pts (xy 245.11 123.952) (xy 231.14 123.952))
+    (stroke (width 0) (type default) (color 0 0 0 0))
+  )
   (wire (pts (xy 117.856 190.5) (xy 115.316 190.5))
     (stroke (width 0) (type default) (color 0 0 0 0))
@@
     (stroke (width 0) (type default) (color 0 0 0 0))
   )
-  (wire (pts (xy 245.11 111.252) (xy 231.14 111.252))
-    (stroke (width 0) (type default) (color 0 0 0 0))
-  )
   (wire (pts (xy 54.356 196.088) (xy 46.736 196.088))
     (stroke (width 0) (type default) (color 0 0 0 0))
@@
     (stroke (width 0) (type default) (color 0 0 0 0))
   )
+  (wire (pts (xy 231.14 111.252) (xy 245.11 111.252))
+    (stroke (width 0) (type default) (color 0 0 0 0))
+  )
   (wire (pts (xy 273.05 187.96) (xy 275.59 187.96))
     (stroke (width 0) (type default) (color 0 0 0 0))
@@
     (stroke (width 0) (type default) (color 0 0 0 0))
   )
-  (wire (pts (xy 245.11 159.512) (xy 231.14 159.512))
-    (stroke (width 0) (type default) (color 0 0 0 0))
-  )
   (wire (pts (xy 232.918 82.042) (xy 232.918 79.502))
     (stroke (width 0) (type default) (color 0 0 0 0))
@@
     (effects (font (size 1.27 1.27)) (justify left bottom))
   )
-  (label "ADC3_IN4" (at 372.618 67.691 0)
+  (label "ADC2_IN3" (at 372.618 67.691 0)
     (effects (font (size 1.27 1.27)) (justify left bottom))
   )
@@
     (effects (font (size 1.27 1.27)) (justify right bottom))
   )
-  (label "ADC1_IN4" (at 372.618 72.771 0)
+  (label "ADC12_IN6" (at 372.618 72.771 0)
     (effects (font (size 1.27 1.27)) (justify left bottom))
   )
@@
     (effects (font (size 1.27 1.27)) (justify right bottom))
   )
-  (label "ADC3_IN7" (at 372.618 65.151 0)
+  (label "ADC5_IN1" (at 372.618 65.151 0)
     (effects (font (size 1.27 1.27)) (justify left bottom))
   )
@@
     (effects (font (size 1.27 1.27)) (justify left bottom))
   )
-  (label "En0" (at 231.14 108.712 0)
+  (label "En9" (at 231.14 108.712 0)
     (effects (font (size 1.27 1.27)) (justify left bottom))
   )
@@
     (effects (font (size 1.27 1.27)) (justify right bottom))
   )
+  (label "ADC12_IN2" (at 231.14 111.252 0)
+    (effects (font (size 1.27 1.27)) (justify left bottom))
+  )
   (label "QUADSPI1_BK1_NCS" (at 227.33 113.792 0)
     (effects (font (size 1.27 1.27)) (justify left bottom))
@@
     (effects (font (size 1.27 1.27)) (justify left bottom))
   )
-  (label "En6" (at 231.14 123.952 0)
-    (effects (font (size 1.27 1.27)) (justify left bottom))
-  )
   (label "ADC2_IN13" (at 231.14 121.412 0)
     (effects (font (size 1.27 1.27)) (justify left bottom))
@@
     (effects (font (size 1.27 1.27)) (justify right bottom))
   )
-  (label "ADC5_IN1" (at 372.618 82.804 0)
+  (label "ADC5_IN13" (at 372.618 82.804 0)
     (effects (font (size 1.27 1.27)) (justify left bottom))
   )
@@
     (effects (font (size 1.27 1.27)) (justify right bottom))
   )
-  (label "En8" (at 231.14 111.252 0)
+  (label "ADC2_IN3" (at 231.14 123.952 0)
     (effects (font (size 1.27 1.27)) (justify left bottom))
   )
@@
     (effects (font (size 1.27 1.27)) (justify left bottom))
   )
-  (label "ADC2_IN12" (at 372.618 60.198 0)
-    (effects (font (size 1.27 1.27)) (justify left bottom))
-  )
-  (label "En9" (at 231.14 118.872 0)
+  (label "ADC3_IN4" (at 372.618 60.198 0)
+    (effects (font (size 1.27 1.27)) (justify left bottom))
+  )
+  (label "En7" (at 231.14 118.872 0)
     (effects (font (size 1.27 1.27)) (justify left bottom))
   )
@@
     (effects (font (size 1.27 1.27)) (justify left bottom))
   )
-  (label "ADC2_IN11" (at 372.618 75.311 0)
-    (effects (font (size 1.27 1.27)) (justify left bottom))
-  )
-  (label "En3" (at 330.2 144.272 180)
+  (label "ADC12_IN2" (at 372.618 75.311 0)
+    (effects (font (size 1.27 1.27)) (justify left bottom))
+  )
+  (label "En0" (at 330.2 144.272 180)
     (effects (font (size 1.27 1.27)) (justify right bottom))
   )
@@
     (effects (font (size 1.27 1.27)) (justify right bottom))
   )
-  (label "ADC5_IN13" (at 372.618 62.611 0)
+  (label "En6" (at 330.2 106.172 180)
+    (effects (font (size 1.27 1.27)) (justify right bottom))
+  )
+  (label "ADC3_IN7" (at 372.618 62.611 0)
     (effects (font (size 1.27 1.27)) (justify left bottom))
   )
@@
     (effects (font (size 1.27 1.27)) (justify right bottom))
   )
-  (label "ADC2_IN12" (at 231.14 159.512 0)
-    (effects (font (size 1.27 1.27)) (justify left bottom))
-  )
   (label "SWDIO" (at 59.055 118.745 180)
     (effects (font (size 1.27 1.27)) (justify right bottom))
   )
-  (label "En7" (at 330.2 137.922 180)
-    (effects (font (size 1.27 1.27)) (justify right bottom))
+  (label "En8" (at 330.2 137.922 180)
+    (effects (font (size 1.27 1.27)) (justify right bottom))
+  )
+  (label "En3" (at 231.14 159.512 0)
+    (effects (font (size 1.27 1.27)) (justify left bottom))
   )
   (label "QUADSPI1_BK1_IO3" (at 166.37 264.795 180)
@@
     (effects (font (size 1.27 1.27)) (justify right bottom))
   )
-  (label "ADC12_IN6" (at 372.618 70.231 0)
-    (effects (font (size 1.27 1.27)) (justify left bottom))
-  )
-  (label "ADC2_IN11" (at 330.2 106.172 180)
-    (effects (font (size 1.27 1.27)) (justify right bottom))
+  (label "ADC1_IN4" (at 372.618 70.231 0)
+    (effects (font (size 1.27 1.27)) (justify left bottom))
   )
   (label "QUADSPI1_BK1_IO0" (at 227.33 156.972 0)

Commit message: Routing complete ex. dip switch
Connections:
- net ANALOG_IN_10: now also U19.11 (PC3); no longer U19.9 (PC1)
- net ANALOG_IN_11: now also U19.9 (PC1); no longer U19.11 (PC3)
- net En10: now also U19.10 (PC2); no longer U19.70 (PD1)
- net En11: now also U19.70 (PD1); no longer U19.10 (PC2)
Changed lines of the file:
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@@
     (effects (font (size 1.27 1.27)) (justify right bottom))
   )
-  (label "ADC12_IN9" (at 372.618 80.391 0)
+  (label "ADC12_IN7" (at 372.618 80.391 0)
     (effects (font (size 1.27 1.27)) (justify left bottom))
   )
@@
     (effects (font (size 1.27 1.27)) (justify right bottom))
   )
-  (label "ADC12_IN7" (at 372.618 77.851 0)
+  (label "ADC12_IN9" (at 372.618 77.851 0)
     (effects (font (size 1.27 1.27)) (justify left bottom))
   )
@@
     (effects (font (size 1.27 1.27)) (justify right bottom))
   )
-  (label "En11" (at 330.2 98.552 180)
+  (label "En10" (at 330.2 98.552 180)
     (effects (font (size 1.27 1.27)) (justify right bottom))
   )
@@
     (effects (font (size 1.27 1.27)) (justify left bottom))
   )
-  (label "En10" (at 330.2 135.382 180)
-    (effects (font (size 1.27 1.27)) (justify right bottom))
-  )
+  (label "En11" (at 330.2 135.382 180)
+    (effects (font (size 1.27 1.27)) (justify right bottom))
+  )

Commit message: UART5 add
Parts:
- added J21: Conn_01x04, Connector_Molex:Molex_SL_171971-0004_1x04_P2.54mm_Vertical, symbol Connector_Generic:Conn_01x04
Connections:
- net +3V3: now also J21.1 (Pin_1)
- net En11: now also U19.72 (PB3); no longer U19.70 (PD1)
- net En8: now also U19.73 (PB4); no longer U19.71 (PD2)
- net GND: now also J21.4 (Pin_4)
- net UART5_TX: now reaches U19.68 (PC12)
- net UART5_TX: now also J21.3 (Pin_3)
- new net UART5_RX: J21.2 (Pin_2), U19.71 (PD2)
- no-connect marks 15 -> 13
Changed lines of the file:
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@@
   (junction (at 115.316 185.42) (diameter 0) (color 0 0 0 0)
   )
-  (no_connect (at 245.11 162.052))
-  (no_connect (at 245.11 164.592))
-  (no_connect (at 316.23 123.952))
   (no_connect (at 245.11 167.132))
   (no_connect (at 128.143 269.875))
@@
   (no_connect (at 245.11 88.392))
   (no_connect (at 245.11 97.282))
+  (no_connect (at 316.23 135.382))
   (no_connect (at 316.23 126.492))
   (no_connect (at 58.293 85.979))
@@
     (stroke (width 0) (type default) (color 0 0 0 0))
   )
+  (wire (pts (xy 201.168 259.08) (xy 201.168 261.62))
+    (stroke (width 0) (type default) (color 0 0 0 0))
+  )
   (wire (pts (xy 59.055 126.365) (xy 47.625 126.365))
     (stroke (width 0) (type default) (color 0 0 0 0))
@@
     (stroke (width 0) (type default) (color 0 0 0 0))
   )
+  (wire (pts (xy 326.263 123.952) (xy 316.23 123.952))
+    (stroke (width 0) (type default) (color 0 0 0 0))
+  )
   (wire (pts (xy 316.23 159.512) (xy 327.914 159.512))
     (stroke (width 0) (type default) (color 0 0 0 0))
@@
     (stroke (width 0) (type default) (color 0 0 0 0))
   )
+  (wire (pts (xy 201.168 250.19) (xy 201.168 251.46))
+    (stroke (width 0) (type default) (color 0 0 0 0))
+  )
   (wire (pts (xy 132.969 51.435) (xy 138.811 51.435))
     (stroke (width 0) (type default) (color 0 0 0 0))
@@
     (stroke (width 0) (type default) (color 0 0 0 0))
   )
+  (wire (pts (xy 193.167 254) (xy 203.2 254))
+    (stroke (width 0) (type default) (color 0 0 0 0))
+  )
   (wire (pts (xy 138.938 104.267) (xy 138.938 105.283))
     (stroke (width 0) (type default) (color 0 0 0 0))
@@
     (stroke (width 0) (type default) (color 0 0 0 0))
   )
-  (wire (pts (xy 330.2 135.382) (xy 316.23 135.382))
-    (stroke (width 0) (type default) (color 0 0 0 0))
-  )
   (wire (pts (xy 156.464 39.751) (xy 162.179 39.751))
     (stroke (width 0) (type default) (color 0 0 0 0))
@@
     (stroke (width 0) (type default) (color 0 0 0 0))
   )
-  (wire (pts (xy 316.23 137.922) (xy 330.2 137.922))
+  (wire (pts (xy 245.11 162.052) (xy 231.14 162.052))
     (stroke (width 0) (type default) (color 0 0 0 0))
   )
@@
     (stroke (width 0) (type default) (color 0 0 0 0))
   )
+  (wire (pts (xy 201.168 259.08) (xy 203.2 259.08))
+    (stroke (width 0) (type default) (color 0 0 0 0))
+  )
   (wire (pts (xy 133.096 177.8) (xy 135.636 176.276))
     (stroke (width 0) (type default) (color 0 0 0 0))
@@
     (stroke (width 0) (type default) (color 0 0 0 0))
   )
+  (wire (pts (xy 201.168 251.46) (xy 203.2 251.46))
+    (stroke (width 0) (type default) (color 0 0 0 0))
+  )
   (wire (pts (xy 241.173 76.962) (xy 241.173 75.692))
     (stroke (width 0) (type default) (color 0 0 0 0))
@@
     (stroke (width 0) (type default) (color 0 0 0 0))
   )
+  (wire (pts (xy 193.167 256.54) (xy 203.2 256.54))
+    (stroke (width 0) (type default) (color 0 0 0 0))
+  )
   (wire (pts (xy 270.51 187.96) (xy 273.05 187.96))
     (stroke (width 0) (type default) (color 0 0 0 0))
@@
     (stroke (width 0) (type default) (color 0 0 0 0))
   )
+  (wire (pts (xy 245.11 164.592) (xy 231.14 164.592))
+    (stroke (width 0) (type default) (color 0 0 0 0))
+  )
   (wire (pts (xy 115.316 187.96) (xy 115.316 190.5))
     (stroke (width 0) (type default) (color 0 0 0 0))
@@
     (stroke (width 0) (type default) (color 0 0 0 0))
   )
+  (wire (pts (xy 326.263 137.922) (xy 316.23 137.922))
+    (stroke (width 0) (type default) (color 0 0 0 0))
+  )
   (wire (pts (xy 135.636 163.576) (xy 121.666 163.576))
     (stroke (width 0) (type default) (color 0 0 0 0))
@@
     (effects (font (size 1.27 1.27)) (justify left bottom))
   )
+  (label "En8" (at 231.14 164.592 0)
+    (effects (font (size 1.27 1.27)) (justify left bottom))
+  )
   (label "ADC2_IN13" (at 231.14 121.412 0)
     (effects (font (size 1.27 1.27)) (justify left bottom))
@@
     (effects (font (size 1.27 1.27)) (justify right bottom))
   )
+  (label "UART5_RX" (at 326.263 137.922 180)
+    (effects (font (size 1.27 1.27)) (justify right bottom))
+  )
   (label "MUX1_SEL0" (at 327.279 82.042 180)
     (effects (font (size 1.27 1.27)) (justify right bottom))
@@
     (effects (font (size 1.27 1.27)) (justify left bottom))
   )
+  (label "UART5_TX" (at 326.263 123.952 180)
+    (effects (font (size 1.27 1.27)) (justify right bottom))
+  )
   (label "SWCLK" (at 233.68 144.272 0)
     (effects (font (size 1.27 1.27)) (justify left bottom))
@@
     (effects (font (size 1.27 1.27)) (justify right bottom))
   )
-  (label "En8" (at 330.2 137.922 180)
-    (effects (font (size 1.27 1.27)) (justify right bottom))
+  (label "UART5_TX" (at 193.167 256.54 0)
+    (effects (font (size 1.27 1.27)) (justify left bottom))
+  )
+  (label "En11" (at 231.14 162.052 0)
+    (effects (font (size 1.27 1.27)) (justify left bottom))
   )
   (label "En3" (at 231.14 159.512 0)
@@
     (effects (font (size 1.27 1.27)) (justify right bottom))
   )
+  (label "UART5_RX" (at 193.167 254 0)
+    (effects (font (size 1.27 1.27)) (justify left bottom))
+  )
   (label "STATUS_LED_2" (at 330.2 84.582 180)
     (effects (font (size 1.27 1.27)) (justify right bottom))
@@
   (label "SPI4_NSS3" (at 121.666 153.416 0)
     (effects (font (size 1.27 1.27)) (justify left bottom))
-  )
-  (label "En11" (at 330.2 135.382 180)
-    (effects (font (size 1.27 1.27)) (justify right bottom))
   )
   (label "ADC5_IN2" (at 231.14 131.572 0)
@@
     (pin "1")
   )
+  (symbol (lib_id "power:+3.3V") (at 201.168 250.19 0) (unit 1)
+    (in_bom yes) (on_board yes)
+    (property "Reference" "#PWR099" (id 0) (at 201.168 254 0)
+      (effects (font (size 1.27 1.27)) hide)
+    )
+    (property "Value" "+3.3V" (id 1) (at 201.549 245.7958 0))
+    (property "Footprint" "" (id 2) (at 201.168 250.19 0)
+      (effects (font (size 1.27 1.27)) hide)
+    )
+    (property "Datasheet" "" (id 3) (at 201.168 250.19 0)
+      (effects (font (size 1.27 1.27)) hide)
+    )
+    (pin "1")
+  )
   (symbol (lib_id "power:GND") (at 148.336 196.596 0) (unit 1)
     (in_bom yes) (on_board yes) (fields_autoplaced)
@@
     )
     (property "Datasheet" "" (id 3) (at 39.878 260.858 0)
+      (effects (font (size 1.27 1.27)) hide)
+    )
+    (pin "1")
+  )
+  (symbol (lib_id "power:GND") (at 201.168 261.62 0) (unit 1)
+    (in_bom yes) (on_board yes) (fields_autoplaced)
+    (property "Reference" "#PWR0100" (id 0) (at 201.168 267.97 0)
+      (effects (font (size 1.27 1.27)) hide)
+    )
+    (property "Value" "GND" (id 1) (at 201.168 266.446 0))
+    (property "Footprint" "" (id 2) (at 201.168 261.62 0)
+      (effects (font (size 1.27 1.27)) hide)
+    )
+    (property "Datasheet" "" (id 3) (at 201.168 261.62 0)
       (effects (font (size 1.27 1.27)) hide)
     )
@@
     (pin "2")
   )
+  (symbol (lib_id "Connector_Generic:Conn_01x04") (at 208.28 254 0) (unit 1)
+    (in_bom yes) (on_board yes) (fields_autoplaced)
+    (property "Reference" "J21" (id 0) (at 211.074 253.9999 0)
+      (effects (font (size 1.27 1.27)) (justify left))
+    )
+    (property "Value" "Conn_01x04" (id 1) (at 211.074 256.5399 0)
+      (effects (font (size 1.27 1.27)) (justify left))
+    )
+    (property "Footprint" "Connector_Molex:Molex_SL_171971-0004_1x04_P2.54mm_Vertical" (id 2) (at 208.28 254 0)
+      (effects (font (size 1.27 1.27)) hide)
+    )
+    (property "Datasheet" "~" (id 3) (at 208.28 254 0)
+      (effects (font (size 1.27 1.27)) hide)
+    )
+    (pin "1")
+    (pin "2")
+    (pin "3")
+    (pin "4")
+  )
   (symbol (lib_id "Connector_Generic:Conn_02x04_Odd_Even") (at 50.673 85.979 0) (unit 1)

Commit message: DIP Switch fix
Parts:
- SW3: footprint TXV_Library_Footprints:8_Pin_DIP_Switch -> TXV_Library_Footprints:8_Pin_DIP_Switch_DHA-08T-Q
Changed lines of the file:
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@@
       (effects (font (size 1.27 1.27)) hide)
     )
-    (property "Footprint" "TXV_Library_Footprints:8_Pin_DIP_Switch" (id 2) (at 125.476 180.34 0)
+    (property "Footprint" "TXV_Library_Footprints:8_Pin_DIP_Switch_DHA-08T-Q" (id 2) (at 125.476 180.34 0)
       (effects (font (size 1.27 1.27)) hide)
     )
-    (property "Datasheet" "~" (id 3) (at 125.476 180.34 0)
+    (property "Datasheet" "https://docs.rs-online.com/0a2b/0900766b8140878c.pdf" (id 3) (at 125.476 180.34 0)
       (effects (font (size 1.27 1.27)) hide)
     )

Commit message: WIP
Parts:
- C14: symbol Device:CP -> Device:C_Polarized
- U15: symbol Regulator_Linear:MCP1700-3302E_SOT23 -> Regulator_Linear:MCP1700x-300xxTT
Connections:
- net +3V3 renamed +3.3V

Commit message: Almost ready to be ordered
Parts:
- C14: symbol Device:C_Polarized -> Device:CP
- U15: symbol Regulator_Linear:MCP1700x-300xxTT -> Regulator_Linear:MCP1700-3302E_SOT23
Connections:
- net SPI4_~{CS}8 is gone; now on net SPI4_~{CS}6: U2.3 (I6)
- net SPI4_~{CS}1: now also U2.8 (I1); no longer U2.6 (I3)
- net SPI4_~{CS}3: now also U2.6 (I3); no longer U2.8 (I1)
- net SPI4_~{CS}4: now also U2.5 (I4); no longer U2.9 (I0)
- net SPI4_~{CS}5: now also U2.4 (I5); no longer U2.5 (I4)
- net SPI4_~{CS}6: no longer U2.2 (I7)
- net SPI4_~{CS}7: now also U2.2 (I7); no longer U2.4 (I5)
- net UART5_RX: now also J21.3 (Pin_3); no longer J21.2 (Pin_2)
- net UART5_TX: now also J21.2 (Pin_2); no longer J21.3 (Pin_3)
- net +3.3V renamed +3V3
- new net SPI4_~{CS}0: U2.9 (I0)
Other:
- moved on the sheet: C11, C8, J21, TP1, TP3, U15
