File: 24V_to_5V-12V_SMPS.kicad_sch (KiCad schematic)
At the start: 10 parts, among them U14 TS30041

Commit message: WIP
Parts:
- added TP5: TestPoint, TestPoint:TestPoint_THTPad_D1.0mm_Drill0.5mm, symbol Connector:TestPoint
Connections:
- net Vout: now also TP5.1
Changed lines of the file:
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@@
     (effects (font (size 1.27 1.27)) (justify left bottom))
   )
-  (text "Vout = 0.9 * (1 + Rtop / Rbot)" (at 175.26 91.44 0)
+  (text "Vout = 0.9 * (1 + Rtop / Rbot)" (at 179.705 89.662 0)
     (effects (font (size 1.27 1.27)) (justify left bottom))
   )
@@
     (pin "2")
   )
+  (symbol (lib_id "Connector:TestPoint") (at 176.53 96.52 0) (unit 1)
+    (in_bom yes) (on_board yes) (fields_autoplaced)
+    (property "Reference" "TP5" (id 0) (at 178.308 93.2179 0)
+      (effects (font (size 1.27 1.27)) (justify left))
+    )
+    (property "Value" "TestPoint" (id 1) (at 175.0568 93.5482 0)
+      (effects (font (size 1.27 1.27)) (justify right) hide)
+    )
+    (property "Footprint" "TestPoint:TestPoint_THTPad_D1.0mm_Drill0.5mm" (id 2) (at 181.61 96.52 0)
+      (effects (font (size 1.27 1.27)) hide)
+    )
+    (property "Datasheet" "~" (id 3) (at 181.61 96.52 0)
+      (effects (font (size 1.27 1.27)) hide)
+    )
+    (pin "1")
+  )
   (symbol (lib_id "Device:C") (at 193.04 114.3 180) (unit 1)

Commit message: Added Servo Config
Parts:
- F25: footprint TXV_Library_Footprints:0805L110SL PPTC Polyfuse Littelfuse -> Fuse:Fuse_0805_2012Metric
Changed lines of the file:
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@@
       (effects (font (size 1.27 1.27)) (justify left))
     )
-    (property "Footprint" "TXV_Library_Footprints:0805L110SL PPTC Polyfuse Littelfuse" (id 2) (at 102.87 95.25 0)
+    (property "Footprint" "Fuse:Fuse_0805_2012Metric" (id 2) (at 102.87 95.25 0)
       (effects (font (size 1.27 1.27)) (justify left) hide)
     )
